File: Overview & Details/Powerboard/Powerboard_Activity/Power_Board.sch (KiCad schematic (older format))
At the start: 29 parts

Commit message: powerboard schematic
Parts:
- added C10: 1μF@10V, symbol Device:C
- added C12: 100μF@10V, symbol Device:CP1
- added C13: 47μF@10V, symbol Device:CP1
- added C14: 22μF@10V, symbol Device:CP1
- added C7: 10μF@16V, symbol Device:CP1
- added C9: 82pF, symbol Device:C
- added D5: PMEG2010AEH, symbol Device:D_Schottky
- added J2, J3: Screw_Terminal_01x04, symbol Connector:Screw_Terminal_01x04
- added J4, J5: Screw_Terminal_01x02, symbol Connector:Screw_Terminal_01x02
- added L5: 10μH, symbol Device:L
- added L6: 22μH, symbol Device:L
- added R7: 130kΩ, symbol Device:R_Small_US
- added R8: 300kΩ, symbol Device:R_Small_US
- added U5: MAX735CSA, symbol Power_Board:MAX735CSA-Regulator_Switching
- gave numbers to parts that had none: 29
Connections:
- net +15V: now also J3.1 (Pin_1)
- net +36V: now also J2.1 (Pin_1), J2.2 (Pin_2)
- net +5VA: now also C10.1, C13.1, J3.2 (Pin_2), U5.1 (~SHDN), U5.8 (V+)
- net +5VL: now also J4.1 (Pin_1)
- net +5VR: now also J5.1 (Pin_1)
- net -5VA: now also C14.2, J3.4 (Pin_4), L6.2
- net GNDS: now also C10.2, C12.1, C13.2, C14.1, C7.2, C9.2, J2.3 (Pin_3), J2.4 (Pin_4), J3.3 (Pin_3), J4.2 (Pin_2), J5.2 (Pin_2), L5.2, R8.2, U5.6 (GND)
- new net: C7.1, R7.1, U5.2 (Vref)
- new net: R7.2, R8.1, U5.3 (SS)
- new net: C9.1, U5.4 (CC)
- new net: C12.2, D5.2 (A), L6.1, U5.5 (Vout)
- new net: D5.1 (K), L5.1, U5.7 (LX)
Other:
- note added: "+36V DC OUT \nto Audio Board"
- note added: "+5V DC @3A max OUT\nto Left LED Board"
- note added: "+5V DC @3A max OUT\nto Right LED Board"
- note added: "DC Power OUT\nto Audio Board"

Commit message: Pre-board review
Parts:
- removed J1: Barrel_Jack, symbol Connector:Barrel_Jack
- removed J2: Screw_Terminal_01x04, symbol Connector:Screw_Terminal_01x04
- added C15, C16: 100μF, Powerboard:PCR1J101MCL1GS, symbol Device:CP1
- added H1, H2, H3, H4: MountingHole, MountingHole:MountingHole_5.3mm_M5, symbol Mechanical:MountingHole
- added J1: Jack-DC, Powerboard:BarrelJack_Power_2.1x5.5mm_11mmThruHole_PanelMount, symbol Power_Board:Jack-DC
- added J2: Screw_Terminal_01x04, Powerboard:AVX-Wire-To-Board-1x4, symbol Power_Board:Screw_Terminal_01x04
- C1, C3, C4, C8: footprint (none) -> Powerboard:PCR1J101MCL1GS
- C10, C14, C7, C9: footprint (none) -> Capacitor_SMD:C_0805_2012Metric_Pad1.15x1.40mm_HandSolder
- C11, C5: footprint (none) -> Capacitor_Tantalum_SMD:CP_EIA-7361-438_AVX-U_Pad2.18x3.30mm_HandSolder
- C12: footprint (none) -> Capacitor_SMD:C_1210_3225Metric_Pad1.42x2.65mm_HandSolder
- C13: footprint (none) -> Capacitor_SMD:CP_Elec_6.3x5.7
- C2: footprint (none) -> Capacitor_SMD:CP_Elec_10x10
- C6: footprint (none) -> Capacitor_SMD:CP_Elec_8x10
- D1, D2, D3, D4: footprint Package_TO_SOT_SMD:TO-252AA_TabPin4 -> Powerboard:TO-252AA_TabPin4
- D5: footprint (none) -> Diode_SMD:D_SOD-123F
- J3: footprint (none) -> Powerboard:AVX-Wire-To-Board-1x4
- J4, J5: footprint (none) -> Powerboard:AVX-Wire-To-Board-1x2
- L1, L3: footprint (none) -> Powerboard:L_Toroid_Horizontal_D21.8mm_P19.60mm_Bourns_2100
- L2, L4: footprint (none) -> Powerboard:Eaton_CTX100-2-52-R
- L5: footprint (none) -> Powerboard:L_Taiyo-Yuden_NR-10050_9.8x10.0mm_HandSoldering
- L6: footprint (none) -> Powerboard:L_Taiyo-Yuden_NR-60xx_HandSoldering
- R1, R10, R2, R3, R4, R5, R6, R7, R8, R9: footprint (none) -> Resistor_SMD:R_0805_2012Metric_Pad1.15x1.40mm_HandSolder
- U5: footprint (none) -> Package_SO:SOP-8_3.9x4.9mm_P1.27mm
Connections:
- net +36V: now also C15.1, C16.1, J1.2, J2.3 (Pin_2), J2.4 (Pin_1)
- net GNDS: now also C15.2, C16.2, J1.1, J2.1 (Pin_4), J2.2 (ePin_3)
