File: Overview & Details/Powerboard/Powerboard_Activity/Power_Board.sch (KiCad schematic (older format))
At the start: 51 parts, among them J1 Jack-DC, J2 Screw_Terminal_01x04, J3 Screw_Terminal_01x04, J4 Screw_Terminal_01x02, J5 Screw_Terminal_01x02, U1 LM2576S-ADJ, U2 LM2576S-ADJ, U3 LM2576S-ADJ, U4 LM2576S-ADJ, U5 MAX735CSA

Commit message: Finish powerboard design
Parts:
- added R12, R14, R5, R6: 20kΩ, Resistor_SMD:R_0805_2012Metric_Pad1.15x1.40mm_HandSolder, symbol Device:R_Small_US
- J3: renamed from J1; symbol Power_Board:Jack-DC -> Power_Board-rescue:Jack-DC-Power_Board
- J4: renamed from J2; symbol Power_Board:Screw_Terminal_01x04 -> Power_Board-rescue:Screw_Terminal_01x04-Power_Board
- U4: renamed from U5; symbol Power_Board:MAX735CSA-Regulator_Switching -> Power_Board-rescue:MAX735CSA-Regulator_Switching-Power_Board
- renumbered C3 to C1, C7 to C10, C1 to C11, C9 to C12, C12 to C13, C6 to C15, C2 to C16, C8 to C2, C15 to C3, C16 to C4, C11 to C6, C10 to C7, C13 to C8, C4 to C9, D2 to D1, D4 to D2, D5 to D3, D3 to D4, D1 to D5, J4 to J1, J5 to J2, J3 to J5, L2 to L1, L4 to L2, L5 to L3, L6 to L4, L3 to L5, L1 to L6, R4 to R1, R1 to R10, R7 to R11, R8 to R13, R10 to R2, R9 to R4, R6 to R7, R2 to R8, R5 to R9, U2 to U1, U4 to U2, U1 to U5
Connections:
- net +5VR: now also C6.1, J2.1 (Pin_1), L2.2, R2.1
- net GNDS: now also R12.1, R14.1, R5.1, R6.1
- net at U3.5 (~ON~/OFF): now also R12.2
- net at U2.5 (~ON~/OFF): now also R6.2
- net at U1.5 (~ON~/OFF): now also R5.2
- net at U5.5 (~ON~/OFF): now also R14.2
